File: 30pin_SIMM_4MB.sch (KiCad schematic (older format))
At the start: 7 parts, among them IC1 4Mx4bit_DRAM, IC2 4Mx4bit_DRAM, IC3 4Mx1bit_DRAM, J1 30pin_SIMM_Edge

Commit message: Added footprints with longer pads for hand soldering
Parts:
- IC1, IC2: footprint 30pin_SIMM:4Mx4bit_DRAM_SOJ-24-26_7.5mm -> 30pin_SIMM:4Mx4bit_DRAM_SOJ-24-26_7.5mm_HandSolder
- IC3: footprint 30pin_SIMM:4Mx1bit_DRAM_SOJ-20-26_7.5mm -> 30pin_SIMM:4Mx1bit_DRAM_SOJ-20-26_7.5mm_HandSolder
Changed lines of the file:
@@
 F 0 "IC1" H 4850 3300 50  0000 C CNN
 F 1 "4Mx4bit_DRAM" H 4850 3200 50  0000 C CNN
-F 2 "30pin_SIMM:4Mx4bit_DRAM_SOJ-24-26_7.5mm" H 3750 3200 50  0001 C CNN
+F 2 "30pin_SIMM:4Mx4bit_DRAM_SOJ-24-26_7.5mm_HandSolder" H 3750 3200 50  0001 C CNN
 F 3 "" H 3750 3200 50  0001 C CNN
 	1    4850 2500
@@
 F 0 "IC2" H 7550 2550 50  0000 L CNN
 F 1 "4Mx4bit_DRAM" H 7758 2505 50  0001 L CNN
-F 2 "30pin_SIMM:4Mx4bit_DRAM_SOJ-24-26_7.5mm" H 7650 2550 50  0001 C CNN
+F 2 "30pin_SIMM:4Mx4bit_DRAM_SOJ-24-26_7.5mm_HandSolder" H 7650 2550 50  0001 C CNN
 F 3 "" H 7650 2550 50  0001 C CNN
 	2    7650 2550
@@
 F 0 "IC3" H 8450 2550 50  0000 L CNN
 F 1 "4Mx1bit_DRAM" H 8750 2650 50  0001 L CNN
-F 2 "30pin_SIMM:4Mx1bit_DRAM_SOJ-20-26_7.5mm" H 8600 2550 50  0001 C CNN
+F 2 "30pin_SIMM:4Mx1bit_DRAM_SOJ-20-26_7.5mm_HandSolder" H 8600 2550 50  0001 C CNN
 F 3 "" H 8600 2550 50  0001 C CNN
 	2    8550 2550
@@
 F 0 "IC3" H 4850 6650 50  0000 C CNN
 F 1 "4Mx1bit_DRAM" H 4850 6550 50  0000 C CNN
-F 2 "30pin_SIMM:4Mx1bit_DRAM_SOJ-20-26_7.5mm" H 3750 6550 50  0001 C CNN
+F 2 "30pin_SIMM:4Mx1bit_DRAM_SOJ-20-26_7.5mm_HandSolder" H 3750 6550 50  0001 C CNN
 F 3 "" H 3750 6550 50  0001 C CNN
 	1    4850 5850
@@
 F 0 "IC1" H 6750 2550 50  0000 C CNN
 F 1 "4Mx4bit_DRAM" H 7150 2500 50  0001 C CNN
-F 2 "30pin_SIMM:4Mx4bit_DRAM_SOJ-24-26_7.5mm" H 5650 3250 50  0001 C CNN
+F 2 "30pin_SIMM:4Mx4bit_DRAM_SOJ-24-26_7.5mm_HandSolder" H 5650 3250 50  0001 C CNN
 F 3 "" H 5650 3250 50  0001 C CNN
 	2    6750 2550
@@
 F 0 "IC2" H 4850 4950 50  0000 C CNN
 F 1 "4Mx4bit_DRAM" H 4850 4850 50  0000 C CNN
-F 2 "30pin_SIMM:4Mx4bit_DRAM_SOJ-24-26_7.5mm" H 4850 4150 50  0001 C CNN
+F 2 "30pin_SIMM:4Mx4bit_DRAM_SOJ-24-26_7.5mm_HandSolder" H 4850 4150 50  0001 C CNN
 F 3 "" H 4850 4150 50  0001 C CNN
 	1    4850 4150

Commit message: Added OSHW Logo to schematic
Changed lines of the file:
@@
 Wire Bus Line
 	4150 1450 4150 6200
+$Comp
+L Graphic:Logo_Open_Hardware_Small #LOGO1
+U 1 1 6045997C
+P 800 7500
+F 0 "#LOGO1" H 800 7775 50  0001 C CNN
+F 1 "Logo_Open_Hardware_Small" H 800 7275 50  0001 C CNN
+F 2 "" H 800 7500 50  0001 C CNN
+F 3 "~" H 800 7500 50  0001 C CNN
+	1    800  7500
+	1    0    0    -1
+$EndComp
 $EndSCHEMATC
